File: mouse_v2.sch (KiCad schematic (older format))
At the start: 0 parts

Commit message: [add] Circuit design almost finished.
Changed lines of the file:
@@
 $Descr A4 11693 8268
 encoding utf-8
-Sheet 1 9
+Sheet 1 14
 Title ""
 Date ""
@@
 F14 "MOTOR21" O L 4550 4800 50
 F15 "MOTOR22" O L 4550 4950 50
-F16 "SPEAKER" O R 6750 4950 50
+F16 "SPEAKER" O R 6750 4450 50
 F17 "TOF1_EN" O R 6750 3200 50
 F18 "TOF2_EN" O R 6750 3350 50
 F19 "TOF3_EN" O R 6750 3500 50
-F20 "IR_ADC1" I R 6750 4500 50
-F21 "IR_ADC2" I R 6750 4600 50
-F22 "IR_LED1" O R 6750 4200 50
-F23 "IR_LED2" O R 6750 4300 50
+F20 "IR_ADC1" I R 6750 3950 50
+F21 "IR_ADC2" I R 6750 4250 50
+F22 "IR_LED1" O R 6750 3800 50
+F23 "IR_LED2" O R 6750 4100 50
+F24 "LED1" O R 6750 5200 50
+F25 "LED2" O R 6750 5050 50
+F26 "LED3" O R 6750 4900 50
+F27 "LED4" O R 6750 4750 50
+F28 "BUTTON" I R 6750 4600 50
 $EndSheet
 $Sheet
@@
 Wire Wire Line
 	4550 3600 2400 3600
+$Sheet
+S 8600 4250 1200 750
+U 5CB44342
+F0 "ir_sensor1" 50
+F1 "schematics/ir_sensor.sch" 50
+F2 "SENSOR_IN" I L 8600 4500 50
+F3 "SENSOR_OUT" O L 8600 4750 50
+$EndSheet
+$Sheet
+S 4600 1000 1900 1100
+U 5CB44455
+F0 "power" 50
+F1 "schematics/power.sch" 50
+$EndSheet
+$Sheet
+S 8600 5300 1200 800
+U 5CC49FA7
+F0 "ir_sensor2" 50
+F1 "schematics/ir_sensor.sch" 50
+F2 "SENSOR_IN" I L 8600 5600 50
+F3 "SENSOR_OUT" O L 8600 5850 50
+$EndSheet
+Wire Wire Line
+	6750 4250 7600 4250
+Wire Wire Line
+	7600 5850 8600 5850
+Wire Wire Line
+	8600 5600 7700 5600
+Wire Wire Line
+	7700 4100 6750 4100
+Wire Wire Line
+	6750 3950 7800 3950
+Wire Wire Line
+	7800 4750 8600 4750
+Wire Wire Line
+	8600 4500 7900 4500
+Wire Wire Line
+	7900 3800 6750 3800
+$Sheet
+S 5050 5600 1700 1100
+U 5CC71EB7
+F0 "user_interface" 50
+F1 "schematics/user_interface.sch" 50
+F2 "LED1" I R 6750 5700 50
+F3 "LED2" I R 6750 5850 50
+F4 "LED3" I R 6750 6000 50
+F5 "LED4" I R 6750 6150 50
+F6 "SPEAKER" I R 6750 6450 50
+F7 "BUTTON" O R 6750 6300 50
+$EndSheet
+Wire Wire Line
+	7900 3800 7900 4500
+Wire Wire Line
+	7800 3950 7800 4750
+Wire Wire Line
+	7700 4100 7700 5600
+Wire Wire Line
+	7600 4250 7600 5850
+Wire Wire Line
+	6750 4450 7500 4450
+Wire Wire Line
+	7500 6450 6750 6450
+Wire Wire Line
+	6750 4600 7400 4600
+Wire Wire Line
+	7400 6300 6750 6300
+Wire Wire Line
+	6750 6150 7300 6150
+Wire Wire Line
+	7200 6000 6750 6000
+Wire Wire Line
+	6750 5850 7100 5850
+Wire Wire Line
+	6750 5200 7000 5200
+Wire Wire Line
+	7000 5700 6750 5700
+Wire Wire Line
+	7500 4450 7500 6450
+Wire Wire Line
+	7400 4600 7400 6300
+Wire Wire Line
+	7200 4900 7200 6000
+Wire Wire Line
+	7000 5200 7000 5700
+Wire Wire Line
+	6750 5050 7100 5050
+Wire Wire Line
+	7100 5050 7100 5850
+Wire Wire Line
+	6750 4900 7200 4900
+Wire Wire Line
+	7300 4750 7300 6150
+Wire Wire Line
+	6750 4750 7300 4750
+$Sheet
+S 2150 1000 1000 800
+U 5CD09D99
+F0 "amp_battery" 50
+F1 "schematics/amp_battery.sch" 50
+$EndSheet
 $EndSCHEMATC

Commit message: [add] Completed parts placement.
Changed lines of the file:
@@
 $Descr A4 11693 8268
 encoding utf-8
-Sheet 1 14
+Sheet 1 15
 Title ""
 Date ""
@@
 	6750 4750 7300 4750
 $Sheet
-S 2150 1000 1000 800
+S 1200 750  1000 800
 U 5CD09D99
 F0 "amp_battery" 50
 F1 "schematics/amp_battery.sch" 50
 $EndSheet
+$Sheet
+S 1200 1900 1000 700
+U 5CD60484
+F0 "converter" 50
+F1 "schematics/converter.sch" 50
+$EndSheet
 $EndSCHEMATC

Commit message: [add] Completed routing.
Changed lines of the file:
@@
 F25 "LED2" O R 6750 5050 50
 F26 "LED3" O R 6750 4900 50
-F27 "LED4" O R 6750 4750 50
-F28 "BUTTON" I R 6750 4600 50
+F27 "BUTTON" I R 6750 4600 50
 $EndSheet
 $Sheet
@@
 F3 "LED2" I R 6750 5850 50
 F4 "LED3" I R 6750 6000 50
-F5 "LED4" I R 6750 6150 50
-F6 "SPEAKER" I R 6750 6450 50
-F7 "BUTTON" O R 6750 6300 50
+F5 "SPEAKER" I R 6750 6450 50
+F6 "BUTTON" O R 6750 6300 50
 $EndSheet
 Wire Wire Line
@@
 	7400 6300 6750 6300
 Wire Wire Line
-	6750 6150 7300 6150
-Wire Wire Line
 	7200 6000 6750 6000
 Wire Wire Line
@@
 Wire Wire Line
 	6750 4900 7200 4900
-Wire Wire Line
-	7300 4750 7300 6150
-Wire Wire Line
-	6750 4750 7300 4750
 $Sheet
 S 1200 750  1000 800
